Commit message: fixed one wheel not moving, added lidar

File: src/morla/urdf/morla_urdf.xacro (robot description, xacro)
@@ -28,5 +28,5 @@
       <origin xyz="0 0 0" rpy=" 0 0 0"/>
       <geometry>
-        <mesh filename="package://morla/meshes/morla_final1.dae" scale="1 1 1"/>
+        <mesh filename="package://morla/meshes/morla_chassis.dae" scale="1 1 1"/>
       </geometry>
     </visual>
@@ -35,5 +35,5 @@
     <pose>0 0 0 0 0 0</pose>
     <inertial>
-      <mass value="1.35"/>
+      <mass value="5.35"/>
       <origin xyz="0 0 0" rpy="0 0 0"/>
       <inertia
@@ -46,5 +46,5 @@
       <origin xyz="0 0 0" rpy="0 0 0"/>
       <geometry>
-        <mesh filename="package://morla/meshes/wheel1.dae" scale="1 1 1"/>
+        <mesh filename="package://morla/meshes/wheel.dae" scale="1 1 1"/>
         <!--<cylinder radius="0.065" length="0.015"/>-->
       </geometry>
@@ -53,5 +53,5 @@
       <origin xyz="0 0 0" rpy="0 0 0"/>
       <geometry>
-        <mesh filename="package://morla/meshes/wheel1.dae" scale="1 1 1"/>
+        <mesh filename="package://morla/meshes/wheel.dae" scale="1 1 1"/>
         <!--<cylinder radius="0.05" length="0.015"/>-->
       </geometry>
@@ -62,5 +62,5 @@
     <pose>0 0 0 0 0 0</pose>
     <inertial>
-      <mass value="1.35"/>
+      <mass value="5.35"/>
       <origin xyz="0 0 0" rpy="0 0 0"/>
       <inertia
@@ -73,5 +73,5 @@
       <origin xyz="0 0 0" rpy="0 0 0"/>
       <geometry>
-        <mesh filename="package://morla/meshes/wheel1.dae" scale="1 1 1"/>
+        <mesh filename="package://morla/meshes/wheel.dae" scale="1 1 1"/>
         <!--<cylinder radius="0.065" length="0.015"/>-->
       </geometry>
@@ -80,5 +80,5 @@
       <origin xyz="0 0 0" rpy="0 0 0"/>
       <geometry>
-        <mesh filename="package://morla/meshes/wheel1.dae" scale="1 1 1"/>
+        <mesh filename="package://morla/meshes/wheel.dae" scale="1 1 1"/>
         <!--<cylinder radius="0.05" length="0.015"/>-->
       </geometry>
@@ -126,5 +126,5 @@
       <origin xyz="0 0 0" rpy="0 0 0"/>
       <geometry>
-        <box size="0.01 0.01 0.01"/>
+        <box size="0.02 0.02 0.02"/>
         <!--<mesh filename="package://morla/meshes/.dae"/>-->
       </geometry>
@@ -133,5 +133,5 @@
       <origin xyz="0 0 0" rpy="0 0 0"/>
       <geometry>
-        <box size="0.01 0.01 0.01"/>
+        <box size="0.02 0.02 0.02"/>
         <!--<mesh filename="package://morla/meshes/hokuyo.dae"/>-->
       </geometry>
@@ -140,5 +140,5 @@
 <!-- joints -->
   <joint name="LIDAR_joint" type="fixed">
-    <origin xyz="0 0 0.1" rpy="0 0 0"/>
+    <origin xyz="0 0 0.08" rpy="0 0 0"/>
     <parent link="morla_chassis"/>
     <child link="LIDAR"/>
@@ -148,5 +148,5 @@
      <child link="right_wheel"/>
      <parent link="morla_chassis"/>
-     <axis xyz="0 0 1" rpy="0 0 0"/>
+     <axis xyz="1 0 0" rpy="0 0 0"/>
      <limit effort="10000" velocity="1000"/>
      <dynamics damping="1.0" friction="1.0"/>
@@ -156,5 +156,5 @@
      <child link="left_wheel"/>
      <parent link="morla_chassis"/>
-     <axis xyz="1 0 0" rpy="0 0 0"/>
+     <axis xyz="-1 0 0" rpy="0 0 0"/>
      <limit effort="10000" velocity="1000"/>
      <dynamics damping="1.0" friction="1.0"/>
@@ -164,5 +164,5 @@
     <child link="omni_wheel"/>
     <parent link="morla_chassis"/>
-    <axis xyz="1 0 0" rpy="0 0 0"/>
+    <axis xyz="0 0 1" rpy="0 0 0"/>
     <limit effort="10000" velocity="1000"/>
     <dynamics damping="1.0" friction="1.0"/>

Commit message: closes #2 ; Changed collision of robot_footprint in urdf

File: src/morla/urdf/morla_urdf.xacro (robot description, xacro)
@@ -2,4 +2,7 @@
 <robot name="morla" xmlns:xacro="http://www.ros.org/wiki/xacro">
 <xacro:include filename="$(find morla)/urdf/morla_urdf.gazebo" />
+  <material name="black">
+    <color rgba="0 0 0 1"/>
+  </material>
   <link name='robot_footprint'> </link>
   <joint name="robot_footprint_joint" type="fixed">
@@ -22,5 +25,5 @@
       <origin xyz="0 0 0" rpy=" 0 0 0"/>
       <geometry>
-        <box size="0.45469 0.28810 0.089"/>
+        <mesh filename="package://morla/meshes/morla_chassis.dae" scale="1 1 1"/>
       </geometry>
     </collision>

Commit message: Changed link name to work with cartographer

File: src/morla/urdf/morla_urdf.xacro (robot description, xacro)
@@ -5,8 +5,8 @@
     <color rgba="0 0 0 1"/>
   </material>
-  <link name='robot_footprint'> </link>
-  <joint name="robot_footprint_joint" type="fixed">
+  <link name='base_link'> </link>
+  <joint name="base_link_joint" type="fixed">
     <origin xyz="0 0 0" rpy="0 0 0" />
-    <parent link="robot_footprint"/>
+    <parent link="base_link"/>
     <child link="morla_chassis" />
   </joint>
